File: cad/BlackIceMx.sch (EAGLE design)
At the start: 6 parts

Commit message: Updated to BlackEdge library
Parts:
- U$1: device amino:BE-CARRIERSMD -> BlackEdge:BE-CARRIERSMD
- renumbered COMS/DBG to COM/DBG
Changed lines of the file:
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@@
 <part name="MX2" library="con-lsta" deviceset="FE15-2" device=""/>
 <part name="MX3" library="con-lsta" deviceset="FE15-2" device=""/>
-<part name="U$1" library="amino" deviceset="BE-CARRIER" device="SMD" value="BE-CARRIERSMD"/>
+<part name="U$1" library="BlackEdge" deviceset="BE-CARRIER" device="SMD" value="BE-CARRIERSMD"/>
 <part name="+3V1" library="supply1" deviceset="+3V3" device=""/>
 <part name="GND1" library="SparkFun-Aesthetics" deviceset="GND" device=""/>
@@
 <part name="SUPPLY4" library="supply2" deviceset="+5V" device=""/>
 <part name="GND49" library="SparkFun-Aesthetics" deviceset="GND" device=""/>
-<part name="COMS/DBG" library="con-lstb" deviceset="MA13-2" device=""/>
+<part name="COM/DBG" library="con-lstb" deviceset="MA13-2" device=""/>
 <part name="FRAME1" library="frames" deviceset="A4L-LOC" device=""/>
 </parts>
@@
 </instance>
 <instance part="GND49" gate="1" x="175.26" y="10.16" smashed="yes"/>
-<instance part="COMS/DBG" gate="G$1" x="154.94" y="33.02" smashed="yes" rot="R180">
+<instance part="COM/DBG" gate="G$1" x="154.94" y="33.02" smashed="yes" rot="R180">
 <attribute name="VALUE" x="158.75" y="53.34" size="1.778" layer="96" rot="R180"/>
 <attribute name="NAME" x="158.75" y="14.478" size="1.778" layer="95" rot="R180"/>
@@
 <wire x1="162.56" y1="40.64" x2="172.72" y2="40.64" width="0.1524" layer="91"/>
 <label x="165.1" y="40.64" size="1.778" layer="95"/>
-<pinref part="COMS/DBG" gate="G$1" pin="8"/>
+<pinref part="COM/DBG" gate="G$1" pin="8"/>
 </segment>
 </net>
@@
 <wire x1="162.56" y1="38.1" x2="172.72" y2="38.1" width="0.1524" layer="91"/>
 <label x="165.1" y="38.1" size="1.778" layer="95"/>
-<pinref part="COMS/DBG" gate="G$1" pin="10"/>
+<pinref part="COM/DBG" gate="G$1" pin="10"/>
 </segment>
 </net>
@@
 </segment>
 <segment>
-<pinref part="COMS/DBG" gate="G$1" pin="12"/>
+<pinref part="COM/DBG" gate="G$1" pin="12"/>
 <wire x1="162.56" y1="35.56" x2="172.72" y2="35.56" width="0.1524" layer="91"/>
 <label x="165.1" y="35.56" size="1.778" layer="95"/>
@@
 <pinref part="SUPPLY4" gate="+5V" pin="+5V"/>
 <wire x1="162.56" y1="48.26" x2="167.64" y2="48.26" width="0.1524" layer="91"/>
-<pinref part="COMS/DBG" gate="G$1" pin="2"/>
+<pinref part="COM/DBG" gate="G$1" pin="2"/>
 <junction x="167.64" y="48.26"/>
 <wire x1="167.64" y1="48.26" x2="172.72" y2="48.26" width="0.1524" layer="91"/>
-<pinref part="COMS/DBG" gate="G$1" pin="4"/>
+<pinref part="COM/DBG" gate="G$1" pin="4"/>
 </segment>
 </net>
@@
 <wire x1="162.56" y1="30.48" x2="172.72" y2="30.48" width="0.1524" layer="91"/>
 <label x="165.1" y="30.48" size="1.778" layer="95"/>
-<pinref part="COMS/DBG" gate="G$1" pin="16"/>
+<pinref part="COM/DBG" gate="G$1" pin="16"/>
 </segment>
 </net>
@@
 </segment>
 <segment>
-<pinref part="COMS/DBG" gate="G$1" pin="18"/>
+<pinref part="COM/DBG" gate="G$1" pin="18"/>
 <wire x1="162.56" y1="27.94" x2="172.72" y2="27.94" width="0.1524" layer="91"/>
 <label x="165.1" y="27.94" size="1.778" layer="95"/>
@@
 </segment>
 <segment>
-<pinref part="COMS/DBG" gate="G$1" pin="15"/>
+<pinref part="COM/DBG" gate="G$1" pin="15"/>
 <wire x1="147.32" y1="30.48" x2="134.62" y2="30.48" width="0.1524" layer="91"/>
 <label x="134.62" y="30.48" size="1.778" layer="95"/>
@@
 <wire x1="147.32" y1="17.78" x2="129.54" y2="17.78" width="0.1524" layer="91"/>
 <junction x="129.54" y="17.78"/>
-<pinref part="COMS/DBG" gate="G$1" pin="6"/>
-<pinref part="COMS/DBG" gate="G$1" pin="9"/>
-<pinref part="COMS/DBG" gate="G$1" pin="14"/>
-<pinref part="COMS/DBG" gate="G$1" pin="20"/>
-<pinref part="COMS/DBG" gate="G$1" pin="25"/>
+<pinref part="COM/DBG" gate="G$1" pin="6"/>
+<pinref part="COM/DBG" gate="G$1" pin="9"/>
+<pinref part="COM/DBG" gate="G$1" pin="14"/>
+<pinref part="COM/DBG" gate="G$1" pin="20"/>
+<pinref part="COM/DBG" gate="G$1" pin="25"/>
 </segment>
 </net>
@@
 <wire x1="147.32" y1="33.02" x2="134.62" y2="33.02" width="0.1524" layer="91"/>
 <label x="134.62" y="33.02" size="1.778" layer="95"/>
-<pinref part="COMS/DBG" gate="G$1" pin="13"/>
+<pinref part="COM/DBG" gate="G$1" pin="13"/>
 </segment>
 <segment>
@@
 <wire x1="147.32" y1="35.56" x2="134.62" y2="35.56" width="0.1524" layer="91"/>
 <label x="134.62" y="35.56" size="1.778" layer="95"/>
-<pinref part="COMS/DBG" gate="G$1" pin="11"/>
+<pinref part="COM/DBG" gate="G$1" pin="11"/>
 </segment>
 <segment>
@@
 <wire x1="147.32" y1="40.64" x2="134.62" y2="40.64" width="0.1524" layer="91"/>
 <label x="134.62" y="40.64" size="1.778" layer="95"/>
-<pinref part="COMS/DBG" gate="G$1" pin="7"/>
+<pinref part="COM/DBG" gate="G$1" pin="7"/>
 </segment>
 <segment>
@@
 <net name="DONE" class="0">
 <segment>
-<pinref part="COMS/DBG" gate="G$1" pin="22"/>
+<pinref part="COM/DBG" gate="G$1" pin="22"/>
 <wire x1="162.56" y1="22.86" x2="172.72" y2="22.86" width="0.1524" layer="91"/>
 <label x="165.1" y="22.86" size="1.778" layer="95"/>
@@
 <net name="SCL" class="0">
 <segment>
-<pinref part="COMS/DBG" gate="G$1" pin="5"/>
+<pinref part="COM/DBG" gate="G$1" pin="5"/>
 <wire x1="147.32" y1="43.18" x2="134.62" y2="43.18" width="0.1524" layer="91"/>
 <label x="134.62" y="43.18" size="1.778" layer="95"/>
@@
 <net name="SDA" class="0">
 <segment>
-<pinref part="COMS/DBG" gate="G$1" pin="3"/>
+<pinref part="COM/DBG" gate="G$1" pin="3"/>
 <wire x1="147.32" y1="45.72" x2="134.62" y2="45.72" width="0.1524" layer="91"/>
 <label x="134.62" y="45.72" size="1.778" layer="95"/>
@@
 <wire x1="147.32" y1="20.32" x2="134.62" y2="20.32" width="0.1524" layer="91"/>
 <label x="134.62" y="20.32" size="1.778" layer="95"/>
-<pinref part="COMS/DBG" gate="G$1" pin="23"/>
+<pinref part="COM/DBG" gate="G$1" pin="23"/>
 </segment>
 <segment>
@@
 <wire x1="147.32" y1="22.86" x2="134.62" y2="22.86" width="0.1524" layer="91"/>
 <label x="134.62" y="22.86" size="1.778" layer="95"/>
-<pinref part="COMS/DBG" gate="G$1" pin="21"/>
+<pinref part="COM/DBG" gate="G$1" pin="21"/>
 </segment>
 <segment>
@@
 <wire x1="147.32" y1="25.4" x2="134.62" y2="25.4" width="0.1524" layer="91"/>
 <label x="134.62" y="25.4" size="1.778" layer="95"/>
-<pinref part="COMS/DBG" gate="G$1" pin="19"/>
+<pinref part="COM/DBG" gate="G$1" pin="19"/>
 </segment>
 <segment>
@@
 <wire x1="162.56" y1="20.32" x2="172.72" y2="20.32" width="0.1524" layer="91"/>
 <label x="165.1" y="20.32" size="1.778" layer="95"/>
-<pinref part="COMS/DBG" gate="G$1" pin="24"/>
-</segment>
-<segment>
+<pinref part="COM/DBG" gate="G$1" pin="24"/>
+</segment>
+<segment>
